Commit message: modify control to work in gz-sim

File: champ_description/urdf/accessories.urdf.xacro (robot description, xacro)
@@ -30,5 +30,5 @@
             <child link="imu_link" />
         </joint>
-        <gazebo reference="imu_link">
+        <!-- <gazebo reference="imu_link">
                 <sensor name="imu_controller" type="imu">
                     <always_on>true</always_on>
@@ -39,16 +39,7 @@
                             <argument>~/out:=data</argument>
                         </ros>
-                        <!-- <updateRate>50.0</updateRate>
-                        <bodyName>imu_link</bodyName>
-                        <topicName>imu/data</topicName>
-                        <accelDrift>0.005 0.005 0.005</accelDrift>
-                        <accelGaussianNoise>0.005 0.005 0.005</accelGaussianNoise>
-                        <rateDrift>0.005 0.005 0.005 </rateDrift>
-                        <rateGaussianNoise>0.005 0.005 0.005 </rateGaussianNoise>
-                        <headingDrift>0.005</headingDrift>
-                        <headingGaussianNoise>0.005</headingGaussianNoise> -->
                     </plugin>
                 </sensor>
-            </gazebo>
+            </gazebo> -->
         <!-- <xacro:include filename="$(find velodyne_description)/urdf/VLP-16.urdf.xacro"/>
         <xacro:VLP-16 parent="${base_name}" name="velodyne" topic="velodyne_points" hz="10" samples="1024" gpu="false" lasers="16" max_range="100">

File: champ_description/urdf/asus_camera.urdf.xacro (robot description, xacro)
@@ -73,5 +73,5 @@
       </xacro:asus_camera_model>
       <!-- ASUS Xtion PRO camera for simulation -->
-      <gazebo reference="${name}_depth_frame">
+      <!-- <gazebo reference="${name}_depth_frame">
         <sensor type="depth" name="${name}">
           <update_rate>20</update_rate>
@@ -88,11 +88,8 @@
             </clip>
           </camera>
-          <!-- Set always_on only sensor, not on plugin -->
           <always_on>1</always_on>
-          <!-- Set update_rate only sensor, not on plugin -->
           <update_rate>30</update_rate>
           <plugin name="${name}_camera_controller" filename="libgazebo_ros_camera.so">
             <ros>
-              <!-- <namespace>custom_ns</namespace> -->
               <argument>custom_camera/image_raw:=${name}/rgb/image_raw</argument>
               <argument>custom_camera/image_depth:=${name}/depth/image_raw</argument>
@@ -107,8 +104,8 @@
                       <durability>volatile</durability>
                       <history>keep_all</history>
-                      <deadline>123</deadline> <!-- milliseconds -->
-                      <lifespan>42</lifespan> <!-- milliseconds -->
+                      <deadline>123</deadline>
+                      <lifespan>42</lifespan>
                       <liveliness>manual_by_topic</liveliness>
-                      <liveliness_lease_duration>1000</liveliness_lease_duration> <!-- milliseconds -->
+                      <liveliness_lease_duration>1000</liveliness_lease_duration>
                   </publisher>
                   <subscription>
@@ -135,8 +132,8 @@
                       <durability>volatile</durability>
                       <history>keep_all</history>
-                      <deadline>123</deadline> <!-- milliseconds -->
-                      <lifespan>42</lifespan> <!-- milliseconds -->
+                      <deadline>123</deadline>
+                      <lifespan>42</lifespan>
                       <liveliness>manual_by_topic</liveliness>
-                      <liveliness_lease_duration>1000</liveliness_lease_duration> <!-- milliseconds -->
+                      <liveliness_lease_duration>1000</liveliness_lease_duration>
                   </publisher>
                   <subscription>
@@ -151,8 +148,8 @@
                       <durability>volatile</durability>
                       <history>keep_all</history>
-                      <deadline>123</deadline> <!-- milliseconds -->
-                      <lifespan>42</lifespan> <!-- milliseconds -->
+                      <deadline>123</deadline>
+                      <lifespan>42</lifespan>
                       <liveliness>manual_by_topic</liveliness>
-                      <liveliness_lease_duration>1000</liveliness_lease_duration> <!-- milliseconds -->
+                      <liveliness_lease_duration>1000</liveliness_lease_duration>
                   </publisher>
                   <subscription>
@@ -163,15 +160,50 @@
               </topic>
             </qos>
-            <!-- Set camera name. If empty, defaults to sensor name (i.e. "sensor_name") -->
-            <!-- <camera_name>custom_camera</camera_name> -->
-            <!-- Set TF frame name. If empty, defaults to link name (i.e. "link_name") -->
             <frame_name>${name}_depth_optical_frame</frame_name>
             <hack_baseline>0.07</hack_baseline>
-            <!-- No need to repeat distortion parameters or to set autoDistortion -->
             <min_depth>0.001</min_depth>
             <max_depth>20.0</max_depth>
           </plugin>
         </sensor>
-      </gazebo>
+      </gazebo> -->
+       <!-- Camera Sensor -->
+      <!-- <gazebo reference="${name}_depth_frame">
+        <sensor name="${name}_rgb_camera" type="camera">
+          <update_rate>30</update_rate>
+          <pose>0 0 0 0 0 0</pose>
+          <camera>
+            <horizontal_fov>1.096</horizontal_fov>
+            <image>
+              <width>640</width>
+              <height>480</height>
+              <format>R8G8B8</format>
+            </image>
+            <clip>
+              <near>0.001</near>
+              <far>20.0</far>
+            </clip>
+          </camera>
+          <always_on>1</always_on>
+          <topic>${name}/rgb/image_raw</topic>
+        </sensor>
+        <sensor name="${name}_depth_camera" type="depth">
+          <update_rate>30</update_rate>
+          <pose>0 0 0 0 0 0</pose>
+          <depth_camera>
+            <horizontal_fov>1.096</horizontal_fov>
+            <image>
+              <width>640</width>
+              <height>480</height>
+              <format>FLOAT32</format>
+            </image>
+            <clip>
+              <near>0.5</near>
+              <far>9.0</far>
+            </clip>
+          </depth_camera>
+          <always_on>1</always_on>
+          <topic>${name}/depth/image_raw</topic>
+        </sensor>
+      </gazebo> -->
     </xacro:macro>
   </robot>

File: champ_description/urdf/hokuyo_utm30lx.urdf.xacro (robot description, xacro)
@@ -59,14 +59,11 @@
             </noise>
           </ray>
-          <plugin name="gazebo_ros_${name}_controller" filename="libgazebo_ros_ray_sensor.so">
+          <!-- <plugin name="gazebo_ros_${name}_controller" filename="libgazebo_ros_ray_sensor.so">
             <ros>
               <argument>~/out:=${ros_topic}</argument>
             </ros>
-            <!-- Set output to sensor_msgs/PointCloud to get same output type as gazebo_ros_block_laser -->
             <output_type>sensor_msgs/LaserScan</output_type>
-            <!-- <frame_name> ommited, will default to block_laser_link -->
-            <!-- min_intensity instead of hokuyoMinIntensity -->
             <min_intensity>100.0</min_intensity>
-          </plugin>
+          </plugin> -->
         </sensor>
       </gazebo>

File: champ_description/urdf/leg.urdf.xacro (robot description, xacro)
@@ -137,7 +137,27 @@
             <origin xyz="0 0 0" rpy="0 0 0" />
         </joint> -->
+        <!-- <ros2_control name="${leg}" type="system">
+            <hardware>
+                <plugin>gazebo_ros2_control/GazeboSystem</plugin>
+            </hardware>
+            <joint name="${leg}_hip_joint">
+                <command_interface name="effort"/>
+                <state_interface name="position"/>
+                <state_interface name="velocity"/>
+            </joint>
+            <joint name="${leg}_upper_leg_joint">
+                <command_interface name="effort"/>
+                <state_interface name="position"/>
+                <state_interface name="velocity"/>
+            </joint>
+            <joint name="${leg}_lower_leg_joint">
+                <command_interface name="effort"/>
+                <state_interface name="position"/>
+                <state_interface name="velocity"/>
+            </joint>
+        </ros2_control>  -->
         <ros2_control name="${leg}" type="system">
             <hardware>
-                <plugin>gazebo_ros2_control/GazeboSystem</plugin>
+                <plugin>ign_ros2_control/IgnitionSystem</plugin>
             </hardware>
             <joint name="${leg}_hip_joint">

Commit message: modify other sensors

File: champ_description/urdf/accessories.urdf.xacro (robot description, xacro)
@@ -30,16 +30,17 @@
             <child link="imu_link" />
         </joint>
-        <!-- <gazebo reference="imu_link">
+        <gazebo reference="imu_link">
                 <sensor name="imu_controller" type="imu">
                     <always_on>true</always_on>
                     <update_rate>50</update_rate>
-                    <plugin name="gazebo_ros_imu_sensor" filename="libgazebo_ros_imu_sensor.so">
+                    <!-- <plugin name="gazebo_ros_imu_sensor" filename="libgazebo_ros_imu_sensor.so">
                         <ros>
                             <namespace>/imu</namespace>
                             <argument>~/out:=data</argument>
                         </ros>
-                    </plugin>
+                    </plugin> -->
+                    <topic>imu/data</topic>
                 </sensor>
-            </gazebo> -->
+            </gazebo>
         <!-- <xacro:include filename="$(find velodyne_description)/urdf/VLP-16.urdf.xacro"/>
         <xacro:VLP-16 parent="${base_name}" name="velodyne" topic="velodyne_points" hz="10" samples="1024" gpu="false" lasers="16" max_range="100">

File: champ_description/urdf/asus_camera.urdf.xacro (robot description, xacro)
@@ -168,5 +168,5 @@
       </gazebo> -->
        <!-- Camera Sensor -->
-      <!-- <gazebo reference="${name}_depth_frame">
+      <gazebo reference="${name}_depth_frame">
         <sensor name="${name}_rgb_camera" type="camera">
           <update_rate>30</update_rate>
@@ -184,4 +184,5 @@
             </clip>
           </camera>
+          <visualize>true</visualize>
           <always_on>1</always_on>
           <topic>${name}/rgb/image_raw</topic>
@@ -202,8 +203,9 @@
             </clip>
           </depth_camera>
+          <visualize>true</visualize>
           <always_on>1</always_on>
           <topic>${name}/depth/image_raw</topic>
         </sensor>
-      </gazebo> -->
+      </gazebo>
     </xacro:macro>
   </robot>

File: champ_description/urdf/champ.urdf.xacro (robot description, xacro)
@@ -66,5 +66,5 @@
         <parent link="world"/>
         <child link="base_link"/>
-      </joint> -->
+    </joint> -->
     <gazebo reference="base_link">
         <material>Gazebo/FlatBlack</material>

File: champ_description/urdf/hokuyo_utm30lx.urdf.xacro (robot description, xacro)
@@ -34,5 +34,5 @@
       </xacro:hokuyo_utm30lx_model>
       <gazebo reference="${name}_frame">
-        <sensor type="ray" name="${name}">
+        <!-- <sensor type="ray" name="${name}">
           <always_on>true</always_on>
           <update_rate>${update_rate}</update_rate>
@@ -59,5 +59,5 @@
             </noise>
           </ray>
-          <!-- <plugin name="gazebo_ros_${name}_controller" filename="libgazebo_ros_ray_sensor.so">
+          <plugin name="gazebo_ros_${name}_controller" filename="libgazebo_ros_ray_sensor.so">
             <ros>
               <argument>~/out:=${ros_topic}</argument>
@@ -65,6 +65,38 @@
             <output_type>sensor_msgs/LaserScan</output_type>
             <min_intensity>100.0</min_intensity>
-          </plugin> -->
-        </sensor>
+          </plugin>
+        </sensor> -->
+      <sensor name="${name}" type="gpu_lidar">
+        <always_on>true</always_on>
+        <update_rate>${update_rate}</update_rate>
+        <pose>0 0 0 0 0 0</pose>
+        <visualize>false</visualize>
+        <topic>${ros_topic}</topic>
+        <lidar>
+          <horizontal>
+            <samples>${ray_count}</samples>
+            <resolution>1</resolution>
+            <min_angle>${min_angle * M_PI/180}</min_angle>
+            <max_angle>${max_angle * M_PI/180}</max_angle>
+          </horizontal>
+          <range>
+            <min>0.2</min>
+            <max>30.0</max>
+            <resolution>0.01</resolution>
+          </range>
+          <noise>
+            <type>gaussian</type>
+            <mean>0.0</mean>
+            <stddev>0.004</stddev>
+          </noise>
+        </lidar>
+        <!-- <plugin name="gz_ros_${name}_controller" filename="gz-sim-ros2-lidar-system">
+          <ros>
+            <remapping>~/out:=${ros_topic}</remapping>
+          </ros>
+          <output_type>sensor_msgs/LaserScan</output_type>
+          <min_intensity>100.0</min_intensity>
+        </plugin> -->
+      </sensor>
       </gazebo>
     </xacro:macro>
@@ -73,5 +105,5 @@
         <xacro:insert_block name="origin" />
       </xacro:hokuyo_utm30lx_model>
-      <gazebo reference="${name}_frame">
+      <!-- <gazebo reference="${name}_frame">
         <sensor type="gpu_ray" name="${name}">
           <update_rate>${update_rate}</update_rate>
@@ -106,5 +138,5 @@
           </plugin>
         </sensor>
-      </gazebo>
+      </gazebo> -->
     </xacro:macro>
 </robot>
